Commit message: modify basic_nodes and basic_urdf pkgs

File: basic_urdf/description/dhpr.urdf.xacro (robot description, xacro)
@@ -35,4 +35,5 @@
       <geometry>
         <box size="0.8 0.6 0.2" />
+        <!-- <mesh filename="package://basic_urdf/meshes/chassis.stl" scale="1.5 1.5 1"/> -->
       </geometry>
     </visual>
@@ -44,5 +45,4 @@
     <parent link="base_link" />
     <axis xyz="0 1 0" rpy="0 0 0" />
-    <limit effort="100" velocity="10" />
     <dynamics damping="1.0" friction="1.0" />
   </joint>
@@ -74,5 +74,4 @@
     <parent link="base_link" />
     <axis xyz="0 1 0" rpy="0 0 0" />
-    <limit effort="100" velocity="10" />
     <dynamics damping="1.0" friction="1.0" />
   </joint>
@@ -98,15 +97,14 @@
     </visual>
   </link>
-  <!-- Joint BaseLink -> LeftWheel -->
-  <joint type="continuous" name="left_wheel_joint">
+  <!-- Joint BaseLink -> RearLeftWheel -->
+  <joint type="continuous" name="rear_left_wheel_joint">
     <origin xyz="-0.25 0.38 0.05" rpy="0 0 0" />
-    <child link="left_wheel" />
+    <child link="rear_left_wheel" />
     <parent link="base_link" />
     <axis xyz="0 1 0" rpy="0 0 0" />
-    <limit effort="100" velocity="10" />
     <dynamics damping="1.0" friction="1.0" />
   </joint>
   <!-- LeftWheel -->
-  <link name='left_wheel'>
+  <link name='rear_left_wheel'>
     <inertial>
       <mass value="5.0" />
@@ -120,5 +118,5 @@
       </geometry>
     </collision>
-    <visual name='left_wheel_visual'>
+    <visual name='rear_left_wheel_visual'>
       <material name="black" />
       <origin xyz="0 0 0" rpy="0 1.5707 1.5707" />
@@ -128,15 +126,14 @@
     </visual>
   </link>
-  <!-- Joint BaseLink -> RightWheel -->
-  <joint type="continuous" name="right_wheel_joint">
+  <!-- Joint BaseLink -> RearRightWheel -->
+  <joint type="continuous" name="rear_right_wheel_joint">
     <origin xyz="-0.25 -0.38 0.05" rpy="0 0 0" />
-    <child link="right_wheel" />
+    <child link="rear_right_wheel" />
     <parent link="base_link" />
     <axis xyz="0 1 0" rpy="0 0 0" />
-    <limit effort="100" velocity="10" />
     <dynamics damping="1.0" friction="1.0" />
   </joint>
   <!-- RightWheel -->
-  <link name='right_wheel'>
+  <link name='rear_right_wheel'>
     <inertial>
       <mass value="5.0" />
@@ -150,5 +147,5 @@
       </geometry>
     </collision>
-    <visual name='right_wheel_visual'>
+    <visual name='rear_right_wheel_visual'>
       <material name="black" />
       <origin xyz="0 0 0" rpy="0 1.5707 1.5707" />
@@ -158,40 +155,31 @@
     </visual>
   </link>
-  <!-- Gazebo -->
-  <gazebo reference="front_left_wheel">
-    <mu1>0.2</mu1>
-    <mu2>0.2</mu2>
-    <kp>1000000.0</kp>
-    <kd>100.0</kd>
-    <minDepth>0.0001</minDepth>
-    <maxVel>1.0</maxVel>
-  </gazebo>
-  <gazebo reference="front_right_wheel">
-    <mu1>0.2</mu1>
-    <mu2>0.2</mu2>
-    <kp>1000000.0</kp>
-    <kd>100.0</kd>
-    <minDepth>0.0001</minDepth>
-    <maxVel>1.0</maxVel>
-  </gazebo>
-  <gazebo reference="left_wheel">
-    <mu1>0.2</mu1>
-    <mu2>0.2</mu2>
-    <kp>1000000.0</kp>
-    <kd>100.0</kd>
-    <minDepth>0.0001</minDepth>
-    <maxVel>1.0</maxVel>
-  </gazebo>
-  <gazebo reference="right_wheel">
-    <mu1>0.2</mu1>
-    <mu2>0.2</mu2>
-    <kp>1000000.0</kp>
-    <kd>100.0</kd>
-    <minDepth>0.0001</minDepth>
-    <maxVel>1.0</maxVel>
-  </gazebo>
-  <gazebo reference="base_link">
-    <mu1>0.000002</mu1>
-    <mu2>0.000002</mu2>
-  </gazebo>
+  <!-- Joint BaseLink -> Lidar -->
+  <joint type="fixed" name="lidar_joint">
+    <origin xyz="0.0 0.0 0.2" rpy="0 0 0" />
+    <child link="lidar_link" />
+    <parent link="base_link" />
+  </joint>
+  <!-- Lidar -->
+  <link name='lidar_link'>
+    <inertial>
+      <mass value="0.3" />
+      <origin xyz="0 0 0.075" rpy="0 0 0" />
+      <inertia ixx="0.0013125" ixy="0" ixz="0" iyy="0.0013125" iyz="0" izz="0.0015" />
+    </inertial>
+    <collision>
+      <origin xyz="0 0 0.075" rpy="0 0 0" />
+      <geometry>
+        <cylinder radius="0.10" length="0.15" />
+      </geometry>
+    </collision>
+    <visual name='lidar_link_visual'>
+      <material name="blue" />
+      <origin xyz="0 0 0.075" rpy="0 0 0" />
+      <geometry>
+        <cylinder radius="0.10" length="0.15" />
+        <!-- <mesh filename="package://basic_urdf/meshes/lidar.stl" scale="1 1 0.7" /> -->
+      </geometry>
+    </visual>
+  </link>
 </robot>

Commit message: add ros_gz_bridge

File: basic_urdf/description/dhpr.urdf.xacro (robot description, xacro)
@@ -19,4 +19,5 @@
   <!-- BaseLink -->
   <link name='base_link'>
+    <pose>0 0 0.1 0 0 0</pose>
     <inertial>
       <mass value="15.0" />
@@ -35,5 +36,4 @@
       <geometry>
         <box size="0.8 0.6 0.2" />
-        <!-- <mesh filename="package://basic_urdf/meshes/chassis.stl" scale="1.5 1.5 1"/> -->
       </geometry>
     </visual>
@@ -45,4 +45,5 @@
     <parent link="base_link" />
     <axis xyz="0 1 0" rpy="0 0 0" />
+    <limit effort="100" velocity="10"/>
     <dynamics damping="1.0" friction="1.0" />
   </joint>
@@ -74,4 +75,5 @@
     <parent link="base_link" />
     <axis xyz="0 1 0" rpy="0 0 0" />
+    <limit effort="100" velocity="10"/>
     <dynamics damping="1.0" friction="1.0" />
   </joint>
@@ -103,4 +105,5 @@
     <parent link="base_link" />
     <axis xyz="0 1 0" rpy="0 0 0" />
+    <limit effort="100" velocity="10"/>
     <dynamics damping="1.0" friction="1.0" />
   </joint>
@@ -132,4 +135,5 @@
     <parent link="base_link" />
     <axis xyz="0 1 0" rpy="0 0 0" />
+    <limit effort="100" velocity="10"/>
     <dynamics damping="1.0" friction="1.0" />
   </joint>
@@ -158,6 +162,6 @@
   <joint type="fixed" name="lidar_joint">
     <origin xyz="0.0 0.0 0.2" rpy="0 0 0" />
+    <parent link="base_link" />
     <child link="lidar_link" />
-    <parent link="base_link" />
   </joint>
   <!-- Lidar -->
@@ -165,19 +169,18 @@
     <inertial>
       <mass value="0.3" />
-      <origin xyz="0 0 0.075" rpy="0 0 0" />
+      <origin xyz="0 0 0" rpy="0 0 0" />
       <inertia ixx="0.0013125" ixy="0" ixz="0" iyy="0.0013125" iyz="0" izz="0.0015" />
     </inertial>
     <collision>
-      <origin xyz="0 0 0.075" rpy="0 0 0" />
+      <origin xyz="0 0 0" rpy="0 0 0" />
       <geometry>
-        <cylinder radius="0.10" length="0.15" />
+        <box size="0.15 0.15 0.15" />
       </geometry>
     </collision>
     <visual name='lidar_link_visual'>
       <material name="blue" />
-      <origin xyz="0 0 0.075" rpy="0 0 0" />
+      <origin xyz="0 0 0" rpy="0 0 0" />
       <geometry>
         <cylinder radius="0.10" length="0.15" />
-        <!-- <mesh filename="package://basic_urdf/meshes/lidar.stl" scale="1 1 0.7" /> -->
       </geometry>
     </visual>

Commit message: add 2d and 3d lidar

File: basic_urdf/description/dhpr.urdf.xacro (robot description, xacro)
@@ -13,5 +13,5 @@
   <!-- Joint BaseFootprint -> BaseLink -->
   <joint name="base_footprint_joint" type="fixed">
-    <origin xyz="0 0 0" rpy="0 0 0" />
+    <origin xyz="0 0 0.1" rpy="0 0 0" />
     <parent link="base_footprint" />
     <child link="base_link" />
@@ -161,7 +161,7 @@
   <!-- Joint BaseLink -> Lidar -->
   <joint type="fixed" name="lidar_joint">
-    <origin xyz="0.0 0.0 0.2" rpy="0 0 0" />
+    <origin xyz="0 0 0.25" rpy="0 0 0" />
+    <child link="lidar_link" />
     <parent link="base_link" />
-    <child link="lidar_link" />
   </joint>
   <!-- Lidar -->

Commit message: add new_iot world

File: basic_urdf/description/dhpr.urdf.xacro (robot description, xacro)
@@ -62,5 +62,5 @@
     </collision>
     <visual name='front_left_wheel_visual'>
-      <material name="black" />
+      <material name="orange" />
       <origin xyz="0 0 0" rpy="0 1.5707 1.5707" />
       <geometry>
@@ -92,5 +92,5 @@
     </collision>
     <visual name='front_right_wheel_visual'>
-      <material name="black" />
+      <material name="orange" />
       <origin xyz="0 0 0" rpy="0 1.5707 1.5707" />
       <geometry>
@@ -122,5 +122,5 @@
     </collision>
     <visual name='rear_left_wheel_visual'>
-      <material name="black" />
+      <material name="orange" />
       <origin xyz="0 0 0" rpy="0 1.5707 1.5707" />
       <geometry>
@@ -152,5 +152,5 @@
     </collision>
     <visual name='rear_right_wheel_visual'>
-      <material name="black" />
+      <material name="orange" />
       <origin xyz="0 0 0" rpy="0 1.5707 1.5707" />
       <geometry>

Commit message: updated urdf and added empty world

File: basic_urdf/description/dhpr.urdf.xacro (robot description, xacro)
@@ -23,10 +23,10 @@
       <mass value="15.0" />
       <origin xyz="0 0 0.1" rpy=" 0 0 0" />
-      <xacro:solid_cuboid_inertia m="15.0" l="0.8" w="0.6" h="0.2" />
+      <xacro:solid_cuboid_inertia m="15.0" l="0.8" w="0.7" h="0.2" />
     </inertial>
     <collision name='collision'>
       <origin xyz="0 0 0.1" rpy=" 0 0 0" />
       <geometry>
-        <box size="0.8 0.6 0.2" />
+        <box size="0.8 0.7 0.2" />
       </geometry>
     </collision>
@@ -35,5 +35,5 @@
       <origin xyz="0 0 0.1" rpy=" 0 0 0" />
       <geometry>
-        <box size="0.8 0.6 0.2" />
+        <box size="0.8 0.7 0.2" />
       </geometry>
     </visual>
@@ -58,5 +58,5 @@
       <origin xyz="0 0 0" rpy="0 1.5707 1.5707" />
       <geometry>
-        <cylinder radius="0.15" length="0.15" />
+        <cylinder radius="0.15" length="0.10" />
       </geometry>
     </collision>
@@ -65,5 +65,5 @@
       <origin xyz="0 0 0" rpy="0 1.5707 1.5707" />
       <geometry>
-        <cylinder radius="0.15" length="0.15" />
+        <cylinder radius="0.15" length="0.10" />
       </geometry>
     </visual>
@@ -88,5 +88,5 @@
       <origin xyz="0 0 0" rpy="0 1.5707 1.5707" />
       <geometry>
-        <cylinder radius="0.15" length="0.15" />
+        <cylinder radius="0.15" length="0.10" />
       </geometry>
     </collision>
@@ -95,5 +95,5 @@
       <origin xyz="0 0 0" rpy="0 1.5707 1.5707" />
       <geometry>
-        <cylinder radius="0.15" length="0.15" />
+        <cylinder radius="0.15" length="0.10" />
       </geometry>
     </visual>
@@ -118,5 +118,5 @@
       <origin xyz="0 0 0" rpy="0 1.5707 1.5707" />
       <geometry>
-        <cylinder radius="0.15" length="0.15" />
+        <cylinder radius="0.15" length="0.10" />
       </geometry>
     </collision>
@@ -125,5 +125,5 @@
       <origin xyz="0 0 0" rpy="0 1.5707 1.5707" />
       <geometry>
-        <cylinder radius="0.15" length="0.15" />
+        <cylinder radius="0.15" length="0.10" />
       </geometry>
     </visual>
@@ -148,5 +148,5 @@
       <origin xyz="0 0 0" rpy="0 1.5707 1.5707" />
       <geometry>
-        <cylinder radius="0.15" length="0.15" />
+        <cylinder radius="0.15" length="0.10" />
       </geometry>
     </collision>
@@ -155,5 +155,5 @@
       <origin xyz="0 0 0" rpy="0 1.5707 1.5707" />
       <geometry>
-        <cylinder radius="0.15" length="0.15" />
+        <cylinder radius="0.15" length="0.10" />
       </geometry>
     </visual>
@@ -161,5 +161,5 @@
   <!-- Joint BaseLink -> Lidar -->
   <joint type="fixed" name="lidar_joint">
-    <origin xyz="0 0 0.25" rpy="0 0 0" />
+    <origin xyz="0 0 0.20" rpy="0 0 0" />
     <child link="lidar_link" />
     <parent link="base_link" />
@@ -182,5 +182,5 @@
       <origin xyz="0 0 0" rpy="0 0 0" />
       <geometry>
-        <cylinder radius="0.10" length="0.15" />
+        <cylinder radius="0.13" length="0.10" />
       </geometry>
     </visual>

Commit message: added new world and modified urdf

File: basic_urdf/description/dhpr.urdf.xacro (robot description, xacro)
@@ -62,5 +62,5 @@
     </collision>
     <visual name='front_left_wheel_visual'>
-      <material name="orange" />
+      <material name="black" />
       <origin xyz="0 0 0" rpy="0 1.5707 1.5707" />
       <geometry>
@@ -92,5 +92,5 @@
     </collision>
     <visual name='front_right_wheel_visual'>
-      <material name="orange" />
+      <material name="black" />
       <origin xyz="0 0 0" rpy="0 1.5707 1.5707" />
       <geometry>
@@ -122,5 +122,5 @@
     </collision>
     <visual name='rear_left_wheel_visual'>
-      <material name="orange" />
+      <material name="black" />
       <origin xyz="0 0 0" rpy="0 1.5707 1.5707" />
       <geometry>
@@ -152,5 +152,5 @@
     </collision>
     <visual name='rear_right_wheel_visual'>
-      <material name="orange" />
+      <material name="black" />
       <origin xyz="0 0 0" rpy="0 1.5707 1.5707" />
       <geometry>

Commit message: added nav controller

File: basic_urdf/description/dhpr.urdf.xacro (robot description, xacro)
@@ -41,8 +41,8 @@
   <!-- Joint BaseLink -> FrontLeftWheel -->
   <joint type="continuous" name="front_left_wheel_joint">
-    <origin xyz="0.25 0.38 0.05" rpy="0 0 0" />
+    <origin xyz="0.25 0.38 0.05" rpy="-1.5707963267948966 0 0" />
     <child link="front_left_wheel" />
     <parent link="base_link" />
-    <axis xyz="0 1 0" rpy="0 0 0" />
+    <axis xyz="0 0 1" />
     <limit effort="100" velocity="10"/>
     <dynamics damping="1.0" friction="1.0" />
@@ -52,9 +52,9 @@
     <inertial>
       <mass value="5.0" />
-      <origin xyz="0 0 0" rpy="0 1.5707 1.5707" />
+      <origin xyz="0 0 0" rpy="0 0 0" />
       <inertia ixx="0.014" ixy="0" ixz="0" iyy="0.014" iyz="0" izz="0.025" />
     </inertial>
     <collision>
-      <origin xyz="0 0 0" rpy="0 1.5707 1.5707" />
+      <origin xyz="0 0 0" rpy="0 0 0" />
       <geometry>
         <cylinder radius="0.15" length="0.10" />
@@ -63,5 +63,5 @@
     <visual name='front_left_wheel_visual'>
       <material name="black" />
-      <origin xyz="0 0 0" rpy="0 1.5707 1.5707" />
+      <origin xyz="0 0 0" rpy="0 0 0" />
       <geometry>
         <cylinder radius="0.15" length="0.10" />
@@ -71,8 +71,8 @@
   <!-- Joint BaseLink -> FrontRightWheel -->
   <joint type="continuous" name="front_right_wheel_joint">
-    <origin xyz="0.25 -0.38 0.05" rpy="0 0 0" />
+    <origin xyz="0.25 -0.38 0.05" rpy="1.5707963267948966 0 0" />
     <child link="front_right_wheel" />
     <parent link="base_link" />
-    <axis xyz="0 1 0" rpy="0 0 0" />
+    <axis xyz="0 0 -1" />
     <limit effort="100" velocity="10"/>
     <dynamics damping="1.0" friction="1.0" />
@@ -82,9 +82,9 @@
     <inertial>
       <mass value="5.0" />
-      <origin xyz="0 0 0" rpy="0 1.5707 1.5707" />
+      <origin xyz="0 0 0" rpy="0 0 0" />
       <inertia ixx="0.014" ixy="0" ixz="0" iyy="0.014" iyz="0" izz="0.025" />
     </inertial>
     <collision>
-      <origin xyz="0 0 0" rpy="0 1.5707 1.5707" />
+      <origin xyz="0 0 0" rpy="0 0 0" />
       <geometry>
         <cylinder radius="0.15" length="0.10" />
@@ -93,5 +93,5 @@
     <visual name='front_right_wheel_visual'>
       <material name="black" />
-      <origin xyz="0 0 0" rpy="0 1.5707 1.5707" />
+      <origin xyz="0 0 0" rpy="0 0 0" />
       <geometry>
         <cylinder radius="0.15" length="0.10" />
@@ -101,8 +101,8 @@
   <!-- Joint BaseLink -> RearLeftWheel -->
   <joint type="continuous" name="rear_left_wheel_joint">
-    <origin xyz="-0.25 0.38 0.05" rpy="0 0 0" />
+    <origin xyz="-0.25 0.38 0.05" rpy="-1.5707963267948966 0 0" />
     <child link="rear_left_wheel" />
     <parent link="base_link" />
-    <axis xyz="0 1 0" rpy="0 0 0" />
+    <axis xyz="0 0 1" />
     <limit effort="100" velocity="10"/>
     <dynamics damping="1.0" friction="1.0" />
@@ -112,9 +112,9 @@
     <inertial>
       <mass value="5.0" />
-      <origin xyz="0 0 0" rpy="0 1.5707 1.5707" />
+      <origin xyz="0 0 0" rpy="0 0 0" />
       <inertia ixx="0.014" ixy="0" ixz="0" iyy="0.014" iyz="0" izz="0.025" />
     </inertial>
     <collision>
-      <origin xyz="0 0 0" rpy="0 1.5707 1.5707" />
+      <origin xyz="0 0 0" rpy="0 0 0" />
       <geometry>
         <cylinder radius="0.15" length="0.10" />
@@ -123,5 +123,5 @@
     <visual name='rear_left_wheel_visual'>
       <material name="black" />
-      <origin xyz="0 0 0" rpy="0 1.5707 1.5707" />
+      <origin xyz="0 0 0" rpy="0 0 0" />
       <geometry>
         <cylinder radius="0.15" length="0.10" />
@@ -131,8 +131,8 @@
   <!-- Joint BaseLink -> RearRightWheel -->
   <joint type="continuous" name="rear_right_wheel_joint">
-    <origin xyz="-0.25 -0.38 0.05" rpy="0 0 0" />
+    <origin xyz="-0.25 -0.38 0.05" rpy="1.5707963267948966 0 0" />
     <child link="rear_right_wheel" />
     <parent link="base_link" />
-    <axis xyz="0 1 0" rpy="0 0 0" />
+    <axis xyz="0 0 -1" />
     <limit effort="100" velocity="10"/>
     <dynamics damping="1.0" friction="1.0" />
@@ -142,9 +142,9 @@
     <inertial>
       <mass value="5.0" />
-      <origin xyz="0 0 0" rpy="0 1.5707 1.5707" />
+      <origin xyz="0 0 0" rpy="0 0 0" />
       <inertia ixx="0.014" ixy="0" ixz="0" iyy="0.014" iyz="0" izz="0.025" />
     </inertial>
     <collision>
-      <origin xyz="0 0 0" rpy="0 1.5707 1.5707" />
+      <origin xyz="0 0 0" rpy="0 0 0" />
       <geometry>
         <cylinder radius="0.15" length="0.10" />
@@ -153,5 +153,5 @@
     <visual name='rear_right_wheel_visual'>
       <material name="black" />
-      <origin xyz="0 0 0" rpy="0 1.5707 1.5707" />
+      <origin xyz="0 0 0" rpy="0 0 0" />
       <geometry>
         <cylinder radius="0.15" length="0.10" />
@@ -161,10 +161,10 @@
   <!-- Joint BaseLink -> Lidar -->
   <joint type="fixed" name="lidar_joint">
-    <origin xyz="0 0 0.20" rpy="0 0 0" />
-    <child link="lidar_link" />
+    <origin xyz="0 0 0.25" rpy="0 0 0" />
+    <child link="laser_frame" />
     <parent link="base_link" />
   </joint>
   <!-- Lidar -->
-  <link name='lidar_link'>
+  <link name='laser_frame'>
     <inertial>
       <mass value="0.3" />
@@ -175,12 +175,12 @@
       <origin xyz="0 0 0" rpy="0 0 0" />
       <geometry>
-        <box size="0.15 0.15 0.15" />
+        <cylinder radius="0.10" length="0.10" />
       </geometry>
     </collision>
-    <visual name='lidar_link_visual'>
+    <visual name='laser_frame_visual'>
       <material name="blue" />
       <origin xyz="0 0 0" rpy="0 0 0" />
       <geometry>
-        <cylinder radius="0.13" length="0.10" />
+        <cylinder radius="0.10" length="0.10" />
       </geometry>
     </visual>
